File: PCB/Mini D1 Puck.kicad_pcb (KiCad board)
At the start: 2 copper layers, 1 part

Commit message: Kicad PCB
Parts:
- added B: + -, Connector_JST:JST_EH_S2B-EH_1x02_P2.50mm_Horizontal, F.Cu at (181.8, 59.5)
- added C1: 200uf 25v, Capacitor_THT:CP_Radial_D8.0mm_P3.50mm, F.Cu at (192.8, 76.5)
- added D1: PWD LED, LED_THT:LED_D3.0mm_Horizontal_O1.27mm_Z2.0mm, F.Cu at (186.7, 79.5)
- added J1: PinHeader_1x03_P2.54mm_Vertical, Connector_PinHeader_2.54mm:PinHeader_1x03_P2.54mm_Vertical, F.Cu at (180.5, 65.5)
- added M: + -, Connector_JST:JST_EH_S2B-EH_1x02_P2.50mm_Horizontal, F.Cu at (190.8, 59.5)
- added Q1: 2N2222, Package_TO_SOT_THT:TO-92, F.Cu at (194.5, 67.5)
- added Q2: 2n2222, Package_TO_SOT_THT:TO-92, F.Cu at (176.5, 56.5)
- added R1: 1K, Resistor_THT:R_Axial_DIN0204_L3.6mm_D1.6mm_P5.08mm_Horizontal, F.Cu at (197.0, 71.0)
- added R2: 56Ohm, Resistor_THT:R_Axial_DIN0204_L3.6mm_D1.6mm_P5.08mm_Horizontal, F.Cu at (189.0, 71.0)
- added R3: 10K, Resistor_THT:R_Axial_DIN0204_L3.6mm_D1.6mm_P5.08mm_Horizontal, F.Cu at (174.0, 64.5)
- added R4: 20K, Resistor_THT:R_Axial_DIN0204_L3.6mm_D1.6mm_P5.08mm_Horizontal, F.Cu at (171.5, 64.5)
- added R5: 1K, Resistor_THT:R_Axial_DIN0204_L3.6mm_D1.6mm_P5.08mm_Horizontal, F.Cu at (174.0, 67.5)
- added SW1: SW_Slide_SPDT_Angled_CK_OS102011MA1Q, Button_Switch_THT:SW_Slide_SPDT_Angled_CK_OS102011MA1Q, F.Cu at (177.0, 83.0)
- moved U1 48.2 mm to (188.6, 70.2)
- renumbered REF** to U1
Routing:
- net (no net): track 0.00 -> 277.9 mm
Other:
- board outline added: 32 x 36 mm
- board text added: "20250430"
- board text added: "NHD-HP P1"
